File: followbuttons/followbuttons.kicad_pcb (KiCad board)
At the start: 2 copper layers, 20.3 x 128.5 mm, 33 parts, among them J1 EuroPower16, J2 Thonkiconn, J3 Thonkiconn, SW1 SW_SPST, SW2 SW_SPST, U1 TL072, U2 TL072

Commit message: asdf
Other:
- board size 20.3 x 128.5 mm -> 62.7 x 136.6 mm
Changed lines of the file:
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@@
     )
     (stroke (width 0.0498) (type solid)) (fill solid) (layer "F.SilkS"))
+  (gr_circle (center 80.8 51.2725) (end 80.8 52.7725)
+    (stroke (width 0.5) (type default)) (fill none) (layer "Edge.Cuts"))
+  (gr_circle (center 72.2 79) (end 72.2 81.5)
+    (stroke (width 0.5) (type default)) (fill none) (layer "Edge.Cuts"))
+  (gr_circle (center 72.1 87.6225) (end 72.1 90.1225)
+    (stroke (width 0.5) (type default)) (fill none) (layer "Edge.Cuts"))
+  (gr_rect (start 62.4 28.0725) (end 82.719999 156.5725)
+    (stroke (width 0.5) (type default)) (fill none) (layer "Edge.Cuts"))
   (gr_circle (center 26.68 23) (end 26.68 24.6)
+    (stroke (width 0.5) (type default)) (fill none) (layer "Edge.Cuts"))
+  (gr_circle (center 80.79 64.792499) (end 80.79 66.292499)
     (stroke (width 0.5) (type default)) (fill none) (layer "Edge.Cuts"))
   (gr_rect (start 20 20) (end 40.32 148.5)
     (stroke (width 0.5) (type default)) (fill none) (layer "Edge.Cuts"))
+  (gr_circle (center 80.5 138.6725) (end 80.5 140.1725)
+    (stroke (width 0.5) (type default)) (fill none) (layer "Edge.Cuts"))
+  (gr_circle (center 80.9 60.212499) (end 80.9 61.712499)
+    (stroke (width 0.5) (type default)) (fill none) (layer "Edge.Cuts"))
+  (gr_circle (center 76.039999 31.0725) (end 76.039999 32.6725)
+    (stroke (width 0.5) (type default)) (fill none) (layer "Edge.Cuts"))
   (gr_line (start 36.5 138) (end 39.5 138)
     (stroke (width 0.5) (type default)) (layer "Edge.Cuts"))
+  (gr_circle (center 71.58 138.772499) (end 71.58 141.272499)
+    (stroke (width 0.5) (type default)) (fill none) (layer "Edge.Cuts"))
   (gr_circle (center 33.64 23) (end 33.64 24.6)
     (stroke (width 0.5) (type default)) (fill none) (layer "Edge.Cuts"))
   (gr_circle (center 33.64 145.5) (end 33.64 147.1)
+    (stroke (width 0.5) (type default)) (fill none) (layer "Edge.Cuts"))
+  (gr_circle (center 71.6 128.4725) (end 71.6 130.9725)
+    (stroke (width 0.5) (type default)) (fill none) (layer "Edge.Cuts"))
+  (gr_circle (center 69.08 153.5725) (end 69.08 155.1725)
     (stroke (width 0.5) (type default)) (fill none) (layer "Edge.Cuts"))
   (gr_line (start 31.5 29) (end 34.5 29)
@@
   (gr_line (start 26.5 138) (end 29.5 138)
     (stroke (width 0.5) (type default)) (layer "Edge.Cuts"))
+  (gr_circle (center 80.8 69.372499) (end 80.8 70.872499)
+    (stroke (width 0.5) (type default)) (fill none) (layer "Edge.Cuts"))
+  (gr_circle (center 80.8 42.0725) (end 80.8 43.5725)
+    (stroke (width 0.5) (type default)) (fill none) (layer "Edge.Cuts"))
+  (gr_circle (center 72.41 63.246607) (end 72.41 66.746607)
+    (stroke (width 0.5) (type default)) (fill none) (layer "Edge.Cuts"))
+  (gr_circle (center 80.5 142.5725) (end 80.5 144.0725)
+    (stroke (width 0.5) (type default)) (fill none) (layer "Edge.Cuts"))
   (gr_circle (center 26.68 145.5) (end 26.68 147.1)
     (stroke (width 0.5) (type default)) (fill none) (layer "Edge.Cuts"))
   (gr_line (start 31.5 138) (end 34.5 138)
     (stroke (width 0.5) (type default)) (layer "Edge.Cuts"))
+  (gr_circle (center 69.08 31.0725) (end 69.08 32.6725)
+    (stroke (width 0.5) (type default)) (fill none) (layer "Edge.Cuts"))
   (gr_line (start 21.5 138) (end 24.5 138)
     (stroke (width 0.5) (type default)) (layer "Edge.Cuts"))
@@
   (gr_line (start 21.5 29) (end 24.5 29)
     (stroke (width 0.5) (type default)) (layer "Edge.Cuts"))
+  (gr_circle (center 72.41 45.146607) (end 72.41 48.646607)
+    (stroke (width 0.5) (type default)) (fill none) (layer "Edge.Cuts"))
+  (gr_circle (center 80.5 134.7725) (end 80.5 136.272499)
+    (stroke (width 0.5) (type default)) (fill none) (layer "Edge.Cuts"))
+  (gr_circle (center 76.039999 153.5725) (end 76.039999 155.1725)
+    (stroke (width 0.5) (type default)) (fill none) (layer "Edge.Cuts"))
+  (gr_circle (center 80.8 46.6725) (end 80.8 48.1725)
+    (stroke (width 0.5) (type default)) (fill none) (layer "Edge.Cuts"))
   (gr_text "Wis Designs 2023" (at 39.3 137.2) (layer "B.SilkS")
     (effects (font (size 1 1) (thickness 0.15)) (justify left bottom mirror))
