File: transistor_vca/transistor_vca.kicad_pcb (KiCad board)
At the start: 2 copper layers, 20.3 x 128.5 mm, 22 parts, among them J1 EuroPower16, Q1 2N3904, Q2 2N3904, U1 TL072, U2 TL072

Commit message: asdf
Parts:
- JCV1, JIN1, JOUT1: moved to B.Cu
- moved JCV1 144.0 mm to (36.2, 181.6), turned to 180 degrees
- moved JIN1 117.7 mm to (26.4, 165.9), turned to 180 degrees
- moved JOUT1 106.5 mm to (46.6, 165.6), turned to 180 degrees
- moved R13 52.5 mm to (34.2, 72.7), turned to 0 degrees
- moved U1 47.5 mm to (36.3, 86.1), turned to 0 degrees
- moved Q1 44.5 mm to (38.8, 68.7)
- moved Q2 44.5 mm to (38.8, 73.1)
- moved R1 44.5 mm to (26.2, 67.7)
- moved R10 44.5 mm to (30.2, 77.7)
- moved R11 44.5 mm to (34.2, 67.7)
- moved R12 44.5 mm to (34.2, 70.2)
- moved R14 44.5 mm to (34.2, 75.2)
- moved R2 44.5 mm to (26.2, 70.2)
- moved R3 44.5 mm to (26.2, 72.7)
- moved R4 44.5 mm to (26.2, 75.2)
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Routing:
- net Net-(JOUT1-PadT): track 63.9 -> 0.00 mm, vias 1 -> 0
- net Net-(R1-Pad1): track 57.6 -> 15.6 mm, vias 3 -> 0
- net (no net): track 0.00 -> 41.5 mm
- net Net-(JIN1-PadT): track 72.4 -> 31.1 mm
- net Net-(U1B--): track 21.8 -> 59.1 mm, vias 2 -> 0
- net Net-(Q1-B): track 14.5 -> 49.7 mm, vias 2 -> 0
- net Net-(Q1-C): track 31.2 -> 0.00 mm
- net Net-(U1A--): track 40.7 -> 10.0 mm, vias 2 -> 0
- net Net-(Q2-C): track 23.9 -> 0.00 mm
- net Net-(Q1-E): track 16.2 -> 32.3 mm, vias 2 -> 0
- net GND: track 4.23 -> 15.9 mm, vias 4 -> 1
- net -12V: track 85.4 -> 75.9 mm
- net Net-(R10-Pad1): track 18.0 -> 9.57 mm, vias 2 -> 0
- net Net-(U2A-+): track 24.6 -> 19.7 mm, vias 2 -> 0
- net Net-(U2A--): track 27.3 -> 31.2 mm, vias 2 -> 0
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Other:
- board size 20.3 x 128.5 mm -> 30.5 x 128.5 mm
