File: wisseq/wisseq.kicad_pcb (KiCad board)
At the start: 2 copper layers, 30.5 x 128.5 mm, 97 parts, among them J1 EuroPower16, J2 Thonkiconn, J3 Thonkiconn, Q1 2N3904, Q10 2N3904, Q2 2N3904, Q3 2N3904, Q4 2N3904, Q5 2N3904, Q6 2N3904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

Commit message: asdf
Parts:
- removed U5: CD4017BM, Package_SO:SOP-16_4.4x10.4mm_P1.27mm
- J1: moved to F.Cu
- moved D14 112.0 mm to (132.8, 66.8), turned to 0 degrees
- moved D16 111.7 mm to (132.8, 85.7), turned to 0 degrees
- moved D15 111.4 mm to (132.8, 76.3), turned to 0 degrees
- moved R46 96.4 mm to (63.1, 37.9), turned to 0 degrees
- moved J1 91.9 mm to (34.4, 22.7), turned to 0 degrees
- moved D2 90.7 mm to (107.6, 67.0), turned to 0 degrees
- moved D10 86.0 mm to (107.6, 76.5), turned to 0 degrees
- moved R40 84.6 mm to (127.7, 85.7), turned to 0 degrees
- moved R43 84.0 mm to (130.1, 95.2)
- moved R41 82.6 mm to (63.1, 25.4), turned to 0 degrees
- moved D11 82.2 mm to (107.6, 85.9), turned to 0 degrees
- moved Q8 81.9 mm to (123.7, 85.7)
- moved R44 80.5 mm to (126.9, 95.2), turned to 0 degrees
- moved R38 80.4 mm to (127.7, 66.8), turned to 0 degrees
- moved Q6 79.4 mm to (123.7, 66.8)
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Routing:
- net Net-(Q4-E): track 223.9 -> 0.00 mm, vias 2 -> 0
- net Net-(Q8-E): track 106.6 -> 0.00 mm, vias 2 -> 0
- net Net-(Q1-E): track 104.5 -> 0.00 mm
- net GND: track 101.8 -> 0.00 mm, vias 50 -> 0
- net +5V: track 100.5 -> 0.00 mm, vias 4 -> 0
- net Net-(Q2-E): track 93.7 -> 0.00 mm, vias 4 -> 0
- net Net-(Q3-E): track 86.7 -> 0.00 mm, vias 2 -> 0
- net Net-(D2-A): track 82.3 -> 0.00 mm, vias 2 -> 0
- net Net-(D10-A): track 68.4 -> 0.00 mm, vias 2 -> 0
- net Net-(D11-A): track 64.0 -> 0.00 mm, vias 3 -> 0
- net e: track 63.6 -> 0.00 mm, vias 3 -> 0
- net Net-(D12-A): track 63.4 -> 0.00 mm, vias 2 -> 0
- net Net-(D15-A): track 62.1 -> 0.00 mm, vias 4 -> 0
- net Net-(Q6-E): track 60.0 -> 0.00 mm, vias 2 -> 0
- net Net-(D10-K): track 56.5 -> 0.00 mm, vias 2 -> 0
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- removed copper zone on B.Cu, net GND
- removed copper zone on F.Cu, net GND
Other:
- board outline removed
- board text removed: "Wis Designs 2023"
- board text removed: "Wisseq v0.2"
