File: wyw/wyw.kicad_pcb (KiCad board)
At the start: 2 copper layers, 81.3 x 128.5 mm, 73 parts, among them J1 Conn_02x08_Odd_Even, J10 02x03, J11 02x02, J12 02x02, J13 02x03, J14 02x02, J15 02x02, J17 02x12, J18 02x02, J19 02x05, J2 02x05, J20 02x03, J21 02x03, J22 02x03, J23 02x03, J24 02x02, J25 02x03, J26 02x03, J27 02x02, J28 02x02, J29 02x03, J3 02x05, J30 02x02, J31 02x03, J32 02x02, J33 02x02, J34 02x05, J36 02x03, J37 02x02, J38 02x02, J39 02x02, J4 02x02, J40 02x02, J41 Thonkiconn, J46 Thonkiconn, J5 02x02, J51 Thonkiconn, J6 02x02, J7 02x03, J8 02x03, J9 02x02, Q1 2N3906S, Q2 MMBT2222A, U1 NE555DR, U3 TL072, U4 TL072, U5 4017bm, U6 XL13700

Commit message: asdf
Parts:
- added D15: LED_EMERALD, LED_SMD:LED_0201_0603Metric, F.Cu at (45.5, 43.2)
- added D15: LED_EMERALD, LED_SMD:LED_0201_0603Metric, F.Cu at (81.7, 80.0)
- added D15: LED_EMERALD, LED_SMD:LED_0201_0603Metric, F.Cu at (31.5, 63.9)
- added D15: LED_EMERALD, LED_SMD:LED_0201_0603Metric, F.Cu at (31.5, 69.0)
- added D15: LED_EMERALD, LED_SMD:LED_0201_0603Metric, F.Cu at (31.5, 77.5)
- added D15: LED_EMERALD, LED_SMD:LED_0201_0603Metric, F.Cu at (88.0, 79.1)
- added D15: LED_EMERALD, LED_SMD:LED_0201_0603Metric, F.Cu at (39.2, 66.3)
- added D15: LED_EMERALD, LED_SMD:LED_0201_0603Metric, F.Cu at (81.5, 90.7)
- added D15: LED_EMERALD, LED_SMD:LED_0201_0603Metric, F.Cu at (30.4, 55.6)
- added D15: LED_EMERALD, LED_SMD:LED_0201_0603Metric, F.Cu at (38.2, 42.3)
- added D15: LED_EMERALD, LED_SMD:LED_0201_0603Metric, F.Cu at (81.7, 78.2)
- added D15: LED_EMERALD, LED_SMD:LED_0201_0603Metric, F.Cu at (38.2, 44.9)
- added D15: LED_EMERALD, LED_SMD:LED_0201_0603Metric, F.Cu at (31.5, 42.4)
- added D15: LED_EMERALD, LED_SMD:LED_0201_0603Metric, F.Cu at (81.5, 92.5)
- added D15: LED_EMERALD, LED_SMD:LED_0201_0603Metric, F.Cu at (87.9, 91.6)
- added D15: LED_EMERALD, LED_SMD:LED_0201_0603Metric, F.Cu at (31.5, 66.4)
- added D15: LED_EMERALD, LED_SMD:LED_0201_0603Metric, F.Cu at (31.5, 45.0)
- added D15: LED_EMERALD, LED_SMD:LED_0201_0603Metric, F.Cu at (39.2, 68.8)
- added D15: LED_EMERALD, LED_SMD:LED_0201_0603Metric, F.Cu at (30.4, 53.8)
- added D15: LED_EMERALD, LED_SMD:LED_0201_0603Metric, F.Cu at (37.8, 78.4)
- added D15: LED_EMERALD, LED_SMD:LED_0201_0603Metric, F.Cu at (31.5, 79.2)
- added D15: LED_EMERALD, LED_SMD:LED_0201_0603Metric, F.Cu at (31.5, 39.9)
- added D16: LED_RED, LED_SMD:LED_0201_0603Metric, F.Cu at (39.6, 42.3)
- added D16: LED_RED, LED_SMD:LED_0201_0603Metric, F.Cu at (82.3, 90.7)
- added D16: LED_RED, LED_SMD:LED_0201_0603Metric, F.Cu at (32.9, 42.4)
- added D16: LED_RED, LED_SMD:LED_0201_0603Metric, F.Cu at (40.0, 68.8)
- added D16: LED_RED, LED_SMD:LED_0201_0603Metric, F.Cu at (46.2, 43.2)
- added D16: LED_RED, LED_SMD:LED_0201_0603Metric, F.Cu at (32.9, 39.9)
- added D16: LED_RED, LED_SMD:LED_0201_0603Metric, F.Cu at (32.3, 66.4)
- added D16: LED_RED, LED_SMD:LED_0201_0603Metric, F.Cu at (88.6, 91.6)
- added D16: LED_RED, LED_SMD:LED_0201_0603Metric, F.Cu at (32.3, 79.2)
- added D16: LED_RED, LED_SMD:LED_0201_0603Metric, F.Cu at (82.4, 80.0)
- added D16: LED_RED, LED_SMD:LED_0201_0603Metric, F.Cu at (32.3, 77.5)
- added D16: LED_RED, LED_SMD:LED_0201_0603Metric, F.Cu at (32.3, 69.0)
- added D16: LED_RED, LED_SMD:LED_0201_0603Metric, F.Cu at (31.8, 53.8)
- added D16: LED_RED, LED_SMD:LED_0201_0603Metric, F.Cu at (82.4, 78.2)
- added D16: LED_RED, LED_SMD:LED_0201_0603Metric, F.Cu at (40.0, 66.3)
- added D16: LED_RED, LED_SMD:LED_0201_0603Metric, F.Cu at (32.9, 45.0)
- added D16: LED_RED, LED_SMD:LED_0201_0603Metric, F.Cu at (31.8, 55.6)
- added D16: LED_RED, LED_SMD:LED_0201_0603Metric, F.Cu at (88.8, 79.1)
- added D16: LED_RED, LED_SMD:LED_0201_0603Metric, F.Cu at (82.3, 92.5)
- added D16: LED_RED, LED_SMD:LED_0201_0603Metric, F.Cu at (32.3, 63.9)
- added D16: LED_RED, LED_SMD:LED_0201_0603Metric, F.Cu at (39.6, 44.9)
- added D16: LED_RED, LED_SMD:LED_0201_0603Metric, F.Cu at (38.6, 78.4)
- added D21: LED_EMERALD, LED_SMD:LED_0201_0603Metric, F.Cu at (38.6, 54.9)
- added D22: LED_RED, LED_SMD:LED_0201_0603Metric, F.Cu at (37.2, 54.9)
- added D23: LED_EMERALD, LED_SMD:LED_0603_1608Metric, F.Cu at (49.9, 79.0)
- added D24: LED_RED, LED_SMD:LED_0603_1608Metric, F.Cu at (49.9, 77.4)
- added R12: 1k, Resistor_SMD:R_0402_1005Metric, F.Cu at (38.7, 48.5)
- added R13: 1k, Resistor_SMD:R_0603_1608Metric, F.Cu at (51.2, 43.5)
- added R15: 1k, Resistor_SMD:R_0402_1005Metric, F.Cu at (48.3, 50.4)
- added R16: 1k, Resistor_SMD:R_0603_1608Metric, F.Cu at (49.9, 80.6)
- added U2: TL072, Package_SO:SOIC-8_3.9x4.9mm_P1.27mm, F.Cu at (43.4, 49.3)
Connections:
- U6 pad 1: Net-(J14-Pin_3) -> Net-(R13-Pad1)
Routing:
- net Net-(U2A--): vias 0 -> 1
- net Net-(D21-A): vias 0 -> 1
- net GND: vias 17 -> 15
