File: wyw/wyw.kicad_sch (KiCad schematic)
At the start: 73 parts, among them J1 Conn_02x08_Odd_Even, J10 02x03, J11 02x02, J12 02x02, J13 02x03, J14 02x02, J15 02x02, J17 02x12, J18 02x02, J19 02x05, J2 02x05, J20 02x03, J21 02x03, J22 02x03, J23 02x03, J24 02x02, J25 02x03, J26 02x03, J27 02x02, J28 02x02, J29 02x03, J3 02x05, J30 02x02, J31 02x03, J32 02x02, J33 02x02, J34 02x05, J36 02x03, J37 02x02, J38 02x02, J39 02x02, J4 02x02, J40 02x02, J41 Thonkiconn, J46 Thonkiconn, J5 02x02, J51 Thonkiconn, J6 02x02, J7 02x03, J8 02x03, J9 02x02, Q1 2N3906S, Q2 MMBT2222A, U1 NE555DR, U3 TL072, U4 TL072, U5 4017bm, U6 XL13700

Commit message: asdf
Parts:
- added D13, D23: LED_EMERALD, LED_SMD:LED_0603_1608Metric, symbol PCM_EuroRackTools:LED_EMERALD
- added D14, D24: LED_RED, LED_SMD:LED_0603_1608Metric, symbol PCM_EuroRackTools:LED_RED
- added D15, D21: LED_EMERALD, LED_SMD:LED_0201_0603Metric, symbol PCM_EuroRackTools:LED_EMERALD
- added D16, D22: LED_RED, LED_SMD:LED_0201_0603Metric, symbol PCM_EuroRackTools:LED_RED
- added R11, R16: 1k, Resistor_SMD:R_0603_1608Metric, symbol EuroRackTools:1k
- added R12, R15: 1k, Resistor_SMD:R_0402_1005Metric, symbol EuroRackTools:1k
- added R13: 1k, Resistor_SMD:R_0603_1608Metric, symbol PCM_EuroRackTools:1k
- added U2: TL072, Package_SO:SOIC-8_3.9x4.9mm_P1.27mm, symbol PCM_EuroRackTools:TL072
Connections:
- net +12V: now also U2.8 (V+)
- net -12V: now also U2.4 (V-)
- net GND: now also D13.1 (K), D14.2 (A), D15.1 (K), D16.2 (A), D21.1 (K), D22.2 (A), D23.1 (K), D24.2 (A)
- net at J14.3 (Pin_3), J14.4 (Pin_4): now also R13.2; no longer U6.1
- net at J24.1 (Pin_1), J24.2 (Pin_2), J24.3 (Pin_3)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: now also U2.3 (+)
- net at J27.1 (Pin_1), J27.2 (Pin_2), J27.3 (Pin_3)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: now also R16.1
- new net: D23.2 (A), D24.1 (K), R16.2
- new net: D13.2 (A), D14.1 (K), R11.2
- new net: D15.2 (A), D16.1 (K), R12.1
- new net: R12.2, U2.6 (-), U2.7
- new net: D21.2 (A), D22.1 (K), R15.2
- new net: R13.1, U6.1
- new net: R15.1, U2.1, U2.2 (-)
Other:
- moved on the sheet: J14
