File: wyw v2/wyw.kicad_pcb (KiCad board)
At the start: 2 copper layers, 81.3 x 128.5 mm, 129 parts, among them J1 Conn_02x08_Odd_Even, J10 02x02, J11 02x02, J12 02x02, J13 02x02, J14 02x02, J15 02x02, J16 02x05, J17 02x12, J18 02x02, J19 02x05, J2 02x05, J20 02x03, J21 02x03, J22 02x03, J23 02x03, J24 02x07, J3 02x05, J34 02x05, J4 02x02, J41 Thonkiconn, J46 Thonkiconn, J5 02x02, J51 Thonkiconn, J6 02x02, J7 02x02, J8 02x02, J9 02x02, U1 XL13700, U10 NE555DR, U2 TL074, U3 TL074, U4 TL074, U5 4017bm, U6 TL074, U7 TL074, U8 TL074, U9 TL074

Commit message: asdf
Parts:
- added D54: LED_BLUE, LED_SMD:LED_0201_0603Metric, F.Cu at (91.1, 45.3)
- added D55: LED_BLUE, LED_SMD:LED_0201_0603Metric, F.Cu at (84.3, 45.0)
- added D56: LED_BLUE, LED_SMD:LED_0201_0603Metric, F.Cu at (84.7, 51.8)
- added D57: LED_BLUE, LED_SMD:LED_0201_0603Metric, F.Cu at (90.2, 43.9)
- added D58: LED_BLUE, LED_SMD:LED_0201_0603Metric, F.Cu at (89.2, 50.1)
- added D59: LED_BLUE, LED_SMD:LED_0201_0603Metric, F.Cu at (86.2, 42.6)
- added D60: LED_BLUE, LED_SMD:LED_0201_0603Metric, F.Cu at (87.6, 52.7)
- added D61: LED_BLUE, LED_SMD:LED_0201_0603Metric, F.Cu at (89.3, 42.5)
- added J25: 02x02, Connector_PinHeader_2.54mm:PinHeader_2x02_P2.54mm_Vertical_SMD, F.Cu at (61.3, 51.4)
- added J26: 02x03, Connector_PinHeader_2.54mm:PinHeader_2x03_P2.54mm_Vertical_SMD, F.Cu at (59.5, 91.2)
- added R33: 1k, Resistor_SMD:R_0603_1608Metric, F.Cu at (79.9, 56.1)
- added R34: 1k, Resistor_SMD:R_0603_1608Metric, F.Cu at (79.9, 62.3)
- added R35: 1k, Resistor_SMD:R_0603_1608Metric, F.Cu at (70.9, 62.3)
- added R36: 1k, Resistor_SMD:R_0603_1608Metric, F.Cu at (70.9, 56.1)
- added R37: 1k, Resistor_SMD:R_0603_1608Metric, F.Cu at (70.1, 46.7)
- added R38: 1k, Resistor_SMD:R_0603_1608Metric, F.Cu at (70.1, 52.9)
- added R39: 100k, Resistor_SMD:R_0603_1608Metric, F.Cu at (80.5, 52.7)
- added R40: 100k, Resistor_SMD:R_0603_1608Metric, F.Cu at (80.5, 49.7)
- added R41: 100k, Resistor_SMD:R_0603_1608Metric, F.Cu at (80.5, 46.7)
- added R42: 1k, Resistor_SMD:R_0603_1608Metric, F.Cu at (79.0, 52.9)
- added R43: 1k, Resistor_SMD:R_0603_1608Metric, F.Cu at (79.0, 46.7)
- added RV7: R_Potentiometer_Trim_US, Potentiometer_SMD:Potentiometer_Bourns_TC33X_Vertical, F.Cu at (62.1, 98.6)
- added RV8: R_Potentiometer_Trim_US, Potentiometer_SMD:Potentiometer_Bourns_TC33X_Vertical, F.Cu at (56.7, 98.6)
- added U11: TL074, Package_SO:SOIC-14_3.9x8.7mm_P1.27mm, F.Cu at (75.4, 59.2)
- added U12: TL074, Package_SO:SOIC-14_3.9x8.7mm_P1.27mm, F.Cu at (74.6, 49.8)
- added U13: TL074, Package_SO:SOIC-14_3.9x8.7mm_P1.27mm, F.Cu at (59.3, 83.1)
- J16: value 02x05 -> 02x02; footprint Connector_PinHeader_2.54mm:PinHeader_2x05_P2.54mm_Vertical_SMD -> Connector_PinHeader_2.54mm:PinHeader_2x02_P2.54mm_Vertical_SMD
- moved J16 27.0 mm to (61.3, 64.9), turned to 180 degrees
- moved U9 23.0 mm to (61.3, 58.2), turned to 90 degrees
- moved U10 22.6 mm to (96.0, 40.4)
- moved J24 14.0 mm to (90.2, 60.3), turned to 90 degrees
- moved R31 13.0 mm to (99.0, 100.9)
- moved R32 13.0 mm to (94.7, 100.9)
- moved J19 3.52 mm to (61.1, 35.5), turned to 90 degrees
- moved J23 2.65 mm to (44.4, 94.5)
- moved J34 2.01 mm to (28.7, 96.0)
- moved D42 1.61 mm to (76.6, 81.3)
- moved D43 1.61 mm to (78.0, 81.3)
- moved D44 1.61 mm to (78.1, 83.9)
- moved D45 1.61 mm to (76.6, 83.9)
- moved D46 1.61 mm to (85.4, 82.3)
- moved D47 1.61 mm to (83.9, 82.3)
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Connections:
- U9 pad 1: Net-(J16-Pin_2) -> Net-(J16-Pin_4)
- U9 pad 10: Net-(J16-Pin_5) -> Net-(J25-Pin_2)
- U9 pad 12: Net-(J16-Pin_7) -> Net-(J25-Pin_1)
- U9 pad 13: Net-(J16-Pin_8) -> Net-(J25-Pin_3)
- U9 pad 14: Net-(J16-Pin_8) -> Net-(J25-Pin_3)
- U9 pad 2: Net-(J16-Pin_2) -> Net-(J16-Pin_4)
- U9 pad 3: Net-(J16-Pin_1) -> Net-(J16-Pin_2)
- U9 pad 6: Net-(J16-Pin_4) -> Net-(J16-Pin_1)
- U9 pad 7: Net-(J16-Pin_4) -> Net-(J16-Pin_1)
- U9 pad 8: Net-(J16-Pin_6) -> Net-(J25-Pin_4)
- U9 pad 9: Net-(J16-Pin_6) -> Net-(J25-Pin_4)
Other:
- board text added: "--- buffers in ---"
- board text added: "--- buffers out ---"
- board text added: "Hysteresis!"
- board text removed: "Buffers In"
- board text removed: "Buffers Out"

Commit message: almost done with wyw v2
Parts:
- added D62: LED_BLUE, LED_SMD:LED_0201_0603Metric, F.Cu at (145.3, 70.5)
- added D63: LED_RED, LED_SMD:LED_0201_0603Metric, F.Cu at (145.3, 72.3)
- added D64: LED_BLUE, LED_SMD:LED_0201_0603Metric, F.Cu at (145.3, 74.0)
- added D65: LED_RED, LED_SMD:LED_0201_0603Metric, F.Cu at (145.3, 75.8)
- added R44: 1k, Resistor_SMD:R_0603_1608Metric, F.Cu at (148.5, 70.9)
- added R45: 1k, Resistor_SMD:R_0603_1608Metric, F.Cu at (148.5, 73.4)
- turned D20 to 180 degrees
Connections:
- RV7 pad 2: Net-(J26-Pin_2) -> Net-(J26-Pin_4)
- RV8 pad 2: Net-(J26-Pin_1) -> Net-(J26-Pin_3)
- U13 pad 10: Net-(J26-Pin_2) -> Net-(J26-Pin_4)
- U13 pad 12: Net-(J26-Pin_1) -> Net-(J26-Pin_3)
- U13 pad 2: Net-(J26-Pin_3) -> Net-(J26-Pin_1)
- U13 pad 3: Net-(J26-Pin_1) -> Net-(J26-Pin_3)
- U13 pad 5: Net-(J26-Pin_2) -> Net-(J26-Pin_4)
- U13 pad 6: Net-(J26-Pin_4) -> Net-(J26-Pin_2)
- U9 pad 5: Net-(J16-Pin_3) -> Net-(J16-Pin_1)
- U9 pad 6: Net-(J16-Pin_1) -> Net-(J16-Pin_3)
- U9 pad 7: Net-(J16-Pin_1) -> Net-(J16-Pin_3)
Routing:
- net Net-(J24-Pin_10): track 0.00 -> 80.4 mm
- net Net-(J24-Pin_11): track 0.00 -> 63.3 mm, vias 0 -> 2
- net Net-(J9-Pin_1): track 0.00 -> 56.6 mm
- net Net-(J11-Pin_1): track 0.00 -> 53.5 mm
- net Net-(J23-Pin_3): track 0.00 -> 52.3 mm
- net Net-(J23-Pin_5): track 0.00 -> 48.7 mm
- net Net-(J5-Pin_2): track 0.00 -> 47.5 mm, vias 0 -> 3
- net Net-(J23-Pin_1): track 0.00 -> 46.5 mm
- net Net-(J24-Pin_5): track 0.00 -> 45.2 mm
- net Net-(J24-Pin_3): track 0.00 -> 45.1 mm, vias 0 -> 2
- net Net-(J5-Pin_1): track 0.00 -> 44.7 mm, vias 0 -> 3
- net Net-(J24-Pin_7): track 0.00 -> 44.0 mm
- net Net-(J14-Pin_1): track 0.00 -> 39.1 mm, vias 0 -> 2
- net Net-(J12-Pin_2): track 0.00 -> 38.4 mm
- net Net-(J17-Pin_7): track 0.00 -> 37.9 mm, vias 0 -> 2
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