File: wyw v2/wyw.kicad_sch (KiCad schematic)
At the start: 129 parts, among them J1 Conn_02x08_Odd_Even, J10 02x02, J11 02x02, J12 02x02, J13 02x02, J14 02x02, J15 02x02, J16 02x05, J17 02x12, J18 02x02, J19 02x05, J2 02x05, J20 02x03, J21 02x03, J22 02x03, J23 02x03, J24 02x07, J3 02x05, J34 02x05, J4 02x02, J41 Thonkiconn, J46 Thonkiconn, J5 02x02, J51 Thonkiconn, J6 02x02, J7 02x02, J8 02x02, J9 02x02, U1 XL13700, U10 NE555DR, U2 TL074, U3 TL074, U4 TL074, U5 4017bm, U6 TL074, U7 TL074, U8 TL074, U9 TL074

Commit message: asdf
Parts:
- removed J16: 02x05, Connector_PinHeader_2.54mm:PinHeader_2x05_P2.54mm_Vertical_SMD, symbol PCM_EuroRackTools:02x05
- added D54, D55, D56, D57, D58, D59, D60, D61, D62, D64: LED_BLUE, LED_SMD:LED_0201_0603Metric, symbol PCM_EuroRackTools:LED_BLUE_0201
- added D63, D65: LED_RED, LED_SMD:LED_0201_0603Metric, symbol PCM_EuroRackTools:LED_RED_0201
- added J16, J25: 02x02, Connector_PinHeader_2.54mm:PinHeader_2x02_P2.54mm_Vertical_SMD, symbol PCM_EuroRackTools:02x02
- added J26: 02x03, Connector_PinHeader_2.54mm:PinHeader_2x03_P2.54mm_Vertical_SMD, symbol PCM_EuroRackTools:02x03
- added R33, R34, R35, R36, R37, R38, R42, R43, R44, R45: 1k, Resistor_SMD:R_0603_1608Metric, symbol PCM_EuroRackTools:1k_0201
- added R39, R40, R41: 100k, Resistor_SMD:R_0603_1608Metric, symbol PCM_EuroRackTools:100k
- added RV7, RV8: R_Potentiometer_Trim_US, Potentiometer_SMD:Potentiometer_Bourns_TC33X_Vertical, symbol PCM_EuroRackTools:TRIMPOT
- added U11, U12, U13: TL074, Package_SO:SOIC-14_3.9x8.7mm_P1.27mm, symbol PCM_EuroRackTools:TL074
Connections:
- net +12V: now also U11.4 (V+), U12.4 (V+), U13.4 (V+)
- net +5V: now also R41.2
- net -12V: now also U11.11 (V-), U12.11 (V-), U13.11 (V-)
- net GND: now also D54.1 (K), D55.1 (K), D56.1 (K), D57.1 (K), D58.1 (K), D59.1 (K), D60.1 (K), D61.1 (K), D62.1 (K), D63.2 (A), D64.1 (K), D65.2 (A), R39.1, RV7.1, RV8.1
- net at U9.10 (+): now also J25.2 (Pin_2)
- net at U9.8, U9.9 (-): now also J25.4 (Pin_4)
- net at U9.3 (+): now also J16.2 (Pin_2)
- net at U9.1, U9.2 (-): now also J16.4 (Pin_4)
- net at U9.5 (+): now also J16.3 (Pin_3)
- net at U9.6 (-), U9.7: now also J16.1 (Pin_1)
- net at U9.12 (+): now also J25.1 (Pin_1)
- net at U9.13 (-), U9.14: now also J25.3 (Pin_3)
- net at J24.1 (Pin_1), J24.2 (Pin_2), U10.2: now also U11.12 (+)
- net at J24.10 (Pin_10), J24.9 (Pin_9), U10.6: now also U12.3 (+)
- net at J24.11 (Pin_11), J24.12 (Pin_12), U10.5: now also U12.5 (+)
- net at J24.3 (Pin_3), J24.4 (Pin_4), U10.7: now also U11.10 (+)
- net at J24.5 (Pin_5), J24.6 (Pin_6), U10.3: now also U11.3 (+)
- net at J24.7 (Pin_7), J24.8 (Pin_8), U10.4: now also U11.5 (+)
- new net: R44.1, U13.8, U13.9 (-)
- new net: D62.2 (A), D63.1 (K), R44.2
- new net: D56.2 (A), R34.2
- new net: D60.2 (A), R36.2
- new net: D59.2 (A), R42.2
- new net: R42.1, U12.8, U12.9 (-)
- new net: R39.2, R40.1, U12.10 (+)
- new net: D64.2 (A), D65.1 (K), R45.2
- new net: J26.5 (Pin_5), RV8.3, U13.1
- new net: J26.1 (Pin_1), U13.2 (-)
- new net: J26.3 (Pin_3), RV8.2, U13.12 (+), U13.3 (+)
- new net: R33.1, U11.13 (-), U11.14
- new net: D55.2 (A), R33.2
- new net: R40.2, R41.1, U12.12 (+)
- new net: R43.1, U12.13 (-), U12.14
- new net: R35.1, U11.6 (-), U11.7
- new net: D61.2 (A), R43.2
- new net: R34.1, U11.8, U11.9 (-)
- new net: J26.4 (Pin_4), RV7.2, U13.10 (+), U13.5 (+)
- new net: J26.6 (Pin_6), RV7.3, U13.7
- new net: R38.1, U12.6 (-), U12.7
- new net: R45.1, U13.13 (-), U13.14
- new net: D54.2 (A), R37.2
- new net: J26.2 (Pin_2), U13.6 (-)
- new net: D58.2 (A), R35.2
- new net: R37.1, U12.1, U12.2 (-)
- new net: D57.2 (A), R38.2
- new net: R36.1, U11.1, U11.2 (-)
Other:
- moved on the sheet: J24

Commit message: almost done with wyw v2
Connections:
- net at U9.6 (-), U9.7: now also J16.3 (Pin_3); no longer J16.1 (Pin_1)
- net at U9.5 (+): now also J16.1 (Pin_1); no longer J16.3 (Pin_3)
Other:
- moved on the sheet: J16, J25, U9A, U9B, U9C, U9D, U9E
